File: HardwareBoard-Arduino/HardwareBoard-Arduino.kicad_sch (KiCad schematic)
At the start: 23 parts, among them J1 Conn_01x07_Male, J10 Screw_Terminal_01x02, J2 Screw_Terminal_01x02, J3 Conn_01x03_Male, J4 Conn_01x03_Male, J5 Conn_01x03_Male, J6 Conn_01x03_Male, J7 Screw_Terminal_01x02, J8 Screw_Terminal_01x02, J9 Screw_Terminal_01x02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

Commit message: Feat: add assets
Other:
- moved on the sheet: C1, H1, H2, H3, H4, J1, J3, J4, J5, J6, J7
