File: Limit_switch_mgmt/Limit_switch_mgmt.kicad_sch (KiCad schematic)
At the start: 22 parts, among them J1 Screw_Terminal_01x02, J2 Screw_Terminal_01x02, J3 Screw_Terminal_01x02, J4 Screw_Terminal_01x02, J5 Screw_Terminal_01x03, J6 Screw_Terminal_01x02, J7 Screw_Terminal_01x02, J8 Screw_Terminal_01x02, J9 Screw_Terminal_01x02, U1 SN74HCT00N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

Commit message: Feat: add assets
Parts:
- H1: footprint (none) -> MountingHole:MountingHole_3mm
Other:
- moved on the sheet: H2, H3, H4, J1, J3, J6, J8, J9
