File: PawerBoard_&_BAU/PawerBoard_&_BAU.kicad_sch (KiCad schematic)
At the start: 83 parts, among them IC1 MC34167TG, J1 Conn_01x02, J10 Conn_01x02, J11 Conn_01x02, J12 Conn_01x02, J2 XT60-M, J3 Conn_01x02, J4 Conn_01x02, J5 Conn_01x02, J6 Conn_01x02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

Commit message: Feat: add assets
Other:
- moved on the sheet: BMS1, C1, C10, C13, C3, C5, C6, C7, C8, Conn_Standard-Tamiya1, Conn_Standard-Tamiya2, D1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
