File: StepperDriver_board/StepperDriver_board.kicad_sch (KiCad schematic)
At the start: 18 parts, among them J1 Conn_01x02, J2 Conn_01x02, J3 Conn_01x02, J4 Conn_01x04_Male, J5 Conn_01x02, J6 Conn_01x04_Male, J7 Conn_01x02, J9 Conn_01x04_Male

Commit message: Feat: add assets
Other:
- moved on the sheet: H1, H2, H3, H4
